File: hardware/pcb/Blugasm.kicad_sch (KiCad schematic)
At the start: 46 parts, among them J1 PWR, J2 OLED, J3 I2C, J4 SERVO1, J5 PJ-102AH, J6 SERVO2, J7 BATT, Q1 DMG3415U, Q2 Q_NMOS_DGS, SW1 PWR, SW2 PEC11R-4225F-50024, U1 MCP73831-2-OT, U2 MP3V5050GP, U3 MCP6001-OT, U4 AP2112K-3.3

Commit message: assign footprints
Parts:
- D2, D4: footprint (none) -> Diode_SMD:D_SOD-123
- D3: footprint (none) -> Diode_SMD:D_SOD-123F
- J7: footprint (none) -> Connector_JST:JST_PH_B2B-PH-K_1x02_P2.00mm_Vertical
Other:
- sheet Controller ports: added GPIO36/S_VP, GPIO39/S_VN; removed GPIO36, GPIO39
Changed lines of the file:
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@@
       (effects (font (size 1.27 1.27)) (justify right))
     )
-    (property "Footprint" "" (id 2) (at 231.14 35.56 90)
+    (property "Footprint" "Diode_SMD:D_SOD-123" (id 2) (at 231.14 35.56 90)
       (effects (font (size 1.27 1.27)) hide)
     )
@@
     (property "Reference" "D3" (id 0) (at 106.68 157.48 0))
     (property "Value" "MBR120" (id 1) (at 106.68 160.02 0))
-    (property "Footprint" "" (id 2) (at 106.68 162.56 0)
+    (property "Footprint" "Diode_SMD:D_SOD-123F" (id 2) (at 106.68 162.56 0)
       (effects (font (size 1.27 1.27)) hide)
     )
@@
       (effects (font (size 1.27 1.27)) (justify left))
     )
-    (property "Footprint" "" (id 2) (at 273.05 146.05 0)
+    (property "Footprint" "Connector_JST:JST_PH_B2B-PH-K_1x02_P2.00mm_Vertical" (id 2) (at 273.05 146.05 0)
       (effects (font (size 1.27 1.27)) hide)
     )
@@
     (property "Reference" "D2" (id 0) (at 54.9275 26.67 0))
     (property "Value" "D_Schottky" (id 1) (at 54.9275 29.21 0))
-    (property "Footprint" "" (id 2) (at 54.61 33.02 0)
+    (property "Footprint" "Diode_SMD:D_SOD-123" (id 2) (at 54.61 33.02 0)
       (effects (font (size 1.27 1.27)) hide)
     )
@@
       (effects (font (size 1.27 1.27)) (justify left top))
     )
-    (pin "GPIO39" input (at 140.97 95.25 180)
-      (effects (font (size 1.27 1.27)) (justify left))
-    )
-    (pin "GPIO36" input (at 163.83 107.95 0)
-      (effects (font (size 1.27 1.27)) (justify right))
-    )
     (pin "GPIO32" bidirectional (at 163.83 93.98 0)
       (effects (font (size 1.27 1.27)) (justify right))
@@
     )
     (pin "GPIO26{slash}DAC2" bidirectional (at 163.83 88.9 0)
+      (effects (font (size 1.27 1.27)) (justify right))
+    )
+    (pin "GPIO39{slash}S_VN" input (at 140.97 95.25 180)
+      (effects (font (size 1.27 1.27)) (justify left))
+    )
+    (pin "GPIO36{slash}S_VP" input (at 163.83 107.95 0)
       (effects (font (size 1.27 1.27)) (justify right))
     )
@@
     )
     (path "/d6463592-ec12-40dc-937a-000502b14276"
-      (reference "D2") (unit 1) (value "D_Schottky") (footprint "")
+      (reference "D2") (unit 1) (value "D_Schottky") (footprint "Diode_SMD:D_SOD-123")
     )
     (path "/878f9a00-b811-4b0c-9b29-b7a49893baec"
-      (reference "D3") (unit 1) (value "MBR120") (footprint "")
+      (reference "D3") (unit 1) (value "MBR120") (footprint "Diode_SMD:D_SOD-123F")
     )
     (path "/01165b14-91ac-49b5-8c4f-fa6f001712c6"
-      (reference "D4") (unit 1) (value "D_Schottky_Small") (footprint "")
+      (reference "D4") (unit 1) (value "D_Schottky_Small") (footprint "Diode_SMD:D_SOD-123")
     )
     (path "/5f47bf49-c2ad-4b68-8c33-8aceef16f698/a18725a9-6be9-4eb0-90a5-584259d7ce71"
@@
     )
     (path "/916c67c1-194b-4f79-887b-25f5c0b071db"
-      (reference "J7") (unit 1) (value "BATT") (footprint "")
+      (reference "J7") (unit 1) (value "BATT") (footprint "Connector_JST:JST_PH_B2B-PH-K_1x02_P2.00mm_Vertical")
     )
     (path "/5f47bf49-c2ad-4b68-8c33-8aceef16f698/e6d26a4a-c441-4c5b-abdd-8f3996a45c15"
@@
     )
     (path "/5f47bf49-c2ad-4b68-8c33-8aceef16f698/04a411e4-5ee2-44ab-9fe9-4584d9fca4ef"
-      (reference "JP1") (unit 1) (value "SolderJumper_3_Bridged123") (footprint "")
+      (reference "JP1") (unit 1) (value "SolderJumper_3_Bridged123") (footprint "SaawLib:SolderJumper-3_P1.3mm_Bridged123_Pad1.0x1.5mm_NumberLabels")
     )
     (path "/146b9379-334d-46e2-b316-69e53731224f"
