File: hardware/pcb/controller.kicad_sch (KiCad schematic)
At the start: 30 parts, among them J10 JTAG, J11 I2C, J8 USB_B_Micro, J9 ESPFlash, Q3 S8050, Q4 S8050, SW3 RESET, SW4 BOOT, U5 CP2102N-A02-GQFN24, U6 ESP32-WROOM-32D

Commit message: assign footprints
Parts:
- JP1: footprint (none) -> SaawLib:SolderJumper-3_P1.3mm_Bridged123_Pad1.0x1.5mm_NumberLabels
Changed lines of the file:
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@@
       (effects (font (size 1.27 1.27)) hide)
     )
-    (property "Footprint" "" (id 2) (at 218.44 144.78 0)
+    (property "Footprint" "SaawLib:SolderJumper-3_P1.3mm_Bridged123_Pad1.0x1.5mm_NumberLabels" (id 2) (at 218.44 144.78 0)
       (effects (font (size 1.27 1.27)) hide)
     )
